Commit message: redesigned the robot and added colors

File: GoChaseIt/my_robot/urdf/my_robot.xacro (robot description, xacro)
@@ -9,5 +9,5 @@
   </joint>
   <joint type="continuous" name="left_wheel_hinge">
-    <origin xyz="0.05 0.15 -0.185" rpy="0 0 0"/>
+    <origin xyz="0 0.15 0" rpy="0 0 0"/>
     <child link="left_wheel"/>
     <parent link="chassis"/>
@@ -17,5 +17,5 @@
   </joint>
   <joint type="continuous" name="right_wheel_hinge">
-    <origin xyz="0.05 -0.15 -0.185" rpy="0 0 0"/>
+    <origin xyz="0 -0.15 0" rpy="0 0 0"/>
     <child link="right_wheel"/>
     <parent link="chassis"/>
@@ -25,5 +25,5 @@
   </joint>
   <joint type="prismatic" name="left_arm_lift">
-    <origin xyz="0.0 0.05 0.25" rpy="0 0 0"/>
+    <origin xyz="0.0 0.05 0.15" rpy="0 0 0"/>
     <child link="left_arm"/>
     <parent link="chassis"/>
@@ -33,5 +33,5 @@
   </joint>
   <joint type="prismatic" name="right_arm_lift">
-    <origin xyz="0.0 -0.05 0.25" rpy="0 0 0"/>
+    <origin xyz="0.0 -0.05 0.15" rpy="0 0 0"/>
     <child link="right_arm"/>
     <parent link="chassis"/>
@@ -41,5 +41,5 @@
   </joint>
   <joint type="fixed" name="camera_joint">
-    <origin xyz="0.2 0 0" rpy="0 0 0"/>
+    <origin xyz="0.25 0 0" rpy="0 0 0"/>
     <child link="camera"/>
     <parent link="chassis"/>
@@ -47,5 +47,5 @@
   </joint>
   <joint type="fixed" name="hokuyo_joint">
-    <origin xyz="0.15 0 0.25" rpy="0 0 0"/>
+    <origin xyz="0.15 0 0.1" rpy="0 0 0"/>
     <child link="hokuyo"/>
     <parent link="chassis"/>
@@ -66,5 +66,5 @@
       <origin xyz="0 0 0" rpy=" 0 0 0"/>
       <geometry>
-        <box size=".4 .2 .4"/>
+        <cylinder radius="0.3" length="0.1"/>
       </geometry>
     </collision>
@@ -72,20 +72,36 @@
       <origin xyz="0 0 0" rpy=" 0 0 0"/>
       <geometry>
-        <box size=".4 .2 .4"/>
+        <cylinder radius="0.25" length="0.1"/>
+        <material name="red"/>
+      </geometry>
+    </visual>
+    <collision name='back_caster_collision'>
+      <origin xyz="-0.15 0 -0.05" rpy=" 0 0 0"/>
+      <geometry>
+        <sphere radius="0.0499"/>
+      </geometry>
+    </collision>
+    <visual name='back_caster_visual'>
+      <origin xyz="-0.15 0 -0.05" rpy=" 0 0 0"/>
+      <geometry>
+        <sphere radius="0.05"/>
       </geometry>
     </visual>
     <collision name='front_caster_collision'>
-      <origin xyz="-0.1 0 -0.2" rpy=" 0 0 0"/>
-      <geometry>
-        <sphere radius="0.0849"/>
+      <origin xyz="0.15 0 -0.05" rpy=" 0 0 0"/>
+      <geometry>
+        <sphere radius="0.0499"/>
       </geometry>
     </collision>
     <visual name='front_caster_visual'>
-      <origin xyz="-0.1 0 -0.2" rpy=" 0 0 0"/>
-      <geometry>
-        <sphere radius="0.085"/>
-      </geometry>
-    </visual>
-  </link>
+      <origin xyz="0.15 0 -0.05" rpy=" 0 0 0"/>
+      <geometry>
+        <sphere radius="0.05"/>
+      </geometry>
+    </visual>
+  </link>
+  <gazebo reference="chassis">
+    <material>Gazebo/Red</material>
+  </gazebo>
   <link name='left_wheel'>
     <pose>0 0 0 0 1.5707 1.5707</pose>
@@ -112,4 +128,7 @@
     </visual>
   </link>
+  <gazebo reference="left_wheel">
+    <material>Gazebo/Blue</material>
+  </gazebo>
   <link name='right_wheel'>
     <pose>0 0 0 0 1.5707 1.5707</pose>
@@ -136,4 +155,7 @@
     </visual>
   </link>
+  <gazebo reference="right_wheel">
+    <material>Gazebo/Blue</material>
+  </gazebo>
   <link name='left_arm'>
     <pose>0 0 0 0 0 0</pose>
